File: _autosave-CustomKeyboard.kicad_pcb (KiCad board)
At the start: 2 copper layers, 300 x 140 mm, 139 parts, among them J1 USB_C_Receptacle_USB2.0_16P, SW1 SW_Push, U1 ATmega32U4-A, Y1 16MHz

Commit message: started pcb
Parts:
- removed U1: ATmega32U4-A, Package_QFP:TQFP-44_10x10mm_P0.8mm
- moved R2 20.8 mm to (236.5, 115.0)
- moved R3 20.8 mm to (236.5, 113.0)
- moved Y1 16.2 mm to (240.5, 106.0)
- moved C7 14.7 mm to (243.0, 102.0), turned to -90 degrees
- moved C1 12.5 mm to (269.0, 109.5), turned to 0 degrees
Routing:
- net ROW4: track 491.2 -> 400.6 mm
- net ROW3: track 467.2 -> 377.7 mm
- net ROW2: track 455.1 -> 429.9 mm
- net ROW1: track 441.1 -> 417.0 mm
- net ROW0: track 424.7 -> 401.7 mm
- net COL13: track 177.6 -> 162.7 mm
- net Net-(U1-~{RESET}): track 31.0 -> 17.7 mm
- net COL12: track 79.2 -> 66.3 mm
- net COL11: track 131.0 -> 118.3 mm
- net COL10: track 111.0 -> 98.5 mm
- net COL9: track 121.2 -> 109.1 mm
- net Net-(U1-XTAL1): track 0.00 -> 11.2 mm, vias 0 -> 2
- net COL5: track 176.1 -> 166.1 mm
- net COL4: track 175.4 -> 165.6 mm
- net COL3: track 194.5 -> 185.3 mm
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