File: CustomKeyboard.kicad_pcb (KiCad board)
At the start: 2 copper layers, 300 x 140 mm, 139 parts, among them J1 USB_C_Receptacle_USB2.0_16P, SW1 SW_Push, U1 ATmega32U4-A, Y1 16MHz

Commit message: many things changed
Parts:
- removed C1: 1uF, Capacitor_SMD:C_0805_2012Metric
- removed C2, C3: 0.1uF, Capacitor_SMD:C_0805_2012Metric
- removed R1, R4: 10k, Resistor_SMD:R_0805_2012Metric
- removed R2, R3: 22, Resistor_SMD:R_0805_2012Metric
- removed SW1: SW_Push, random-keyboard-parts.pretty-master:SKQG-1155865
- removed Y1: 16MHz, Crystal:Crystal_SMD_3225-4Pin_3.2x2.5mm
- added C10: 1uF, Capacitor_SMD:C_0603_1608Metric, B.Cu at (220.5, 115.4)
- added C11: 100nF, Capacitor_SMD:C_0603_1608Metric, F.Cu at (118.7, 51.5)
- added C12: 1uF, Capacitor_SMD:C_0603_1608Metric, F.Cu at (118.7, 53.1)
- added C13: 100nF, Capacitor_SMD:C_0603_1608Metric, F.Cu at (291.6, 51.2)
- added C14: 1uF, Capacitor_SMD:C_0603_1608Metric, F.Cu at (291.6, 52.9)
- added C15: 100nF, Capacitor_SMD:C_0603_1608Metric, F.Cu at (329.2, 118.7)
- added C16: 1uF, Capacitor_SMD:C_0603_1608Metric, F.Cu at (327.6, 118.7)
- added C17: 10uF, Capacitor_SMD:C_0603_1608Metric, B.Cu at (176.9, 48.8)
- added C18: 10uF, Capacitor_SMD:C_0603_1608Metric, B.Cu at (179.9, 48.8)
- added C19: 100nF, Capacitor_SMD:C_0402_1005Metric, B.Cu at (200.8, 138.9)
- added C20: 4.7uF, Capacitor_SMD:C_0402_1005Metric, B.Cu at (200.8, 137.9)
- added C21: 100nF, Capacitor_SMD:C_0402_1005Metric, B.Cu at (213.2, 144.4)
- added C22: 10nF, Capacitor_SMD:C_0402_1005Metric, B.Cu at (206.1, 147.8)
- added C23: 1uF, Capacitor_SMD:C_0402_1005Metric, B.Cu at (205.1, 147.8)
- added C24: 100nF, Capacitor_SMD:C_0402_1005Metric, B.Cu at (210.8, 136.2)
- added C25: 4.7uF, Capacitor_SMD:C_0402_1005Metric, B.Cu at (211.8, 136.2)
- added C8: 10uF, Capacitor_SMD:C_0603_1608Metric, B.Cu at (201.6, 53.9)
- added C9: 100nF, Capacitor_SMD:C_0603_1608Metric, B.Cu at (222.1, 115.4)
- added D63: LED, LED_SMD:LED_0805_2012Metric, B.Cu at (201.6, 50.2)
- added F1: 500mA, Fuse:Fuse_0603_1608Metric, B.Cu at (214.6, 116.8)
- added F2: Polyfuse_Small, Fuse:Fuse_1206_3216Metric, B.Cu at (198.8, 56.6)
- added J2: Conn_01x04, CustomFootprints:4_Pad_2.54_Exposed, B.Cu at (267.0, 47.1)
- added J3: Conn_01x04, CustomFootprints:4_Pad_2.54_Exposed, F.Cu at (292.0, 47.1)
- added J4: Conn_01x04, CustomFootprints:4_Pad_2.54_Exposed, B.Cu at (332.4, 87.5)
- added J5: Conn_01x04, CustomFootprints:4_Pad_2.54_Exposed, F.Cu at (332.4, 112.5)
- added J6: Conn_01x04, CustomFootprints:4_Pad_2.54_Exposed, B.Cu at (94.1, 47.1)
- added J7: Conn_01x04, CustomFootprints:4_Pad_2.54_Exposed, B.Cu at (119.1, 47.1)
- added R10: 10k, Resistor_SMD:R_0402_1005Metric, B.Cu at (203.7, 112.8)
- added R7: 620, Resistor_SMD:R_0603_1608Metric, B.Cu at (201.6, 52.3)
- added REF**: PinHeader_1x04_P2.54mm_Vertical, Connector_PinHeader_2.54mm:PinHeader_1x04_P2.54mm_Vertical, F.Cu at (115.2, 37.6)
- added REF**: STAB_MX_P_6.25u, PCM_marbastlib-mx:STAB_MX_P_6.25u, F.Cu at (182.1, 145.0)
- added REF**: ConnectorMicromatch-4, ConnectorMicromatch-4, F.Cu at (94.0, 41.0)
- added REF**: ConnectorMicromatch-4, ConnectorMicromatch-4, F.Cu at (267.0, 41.0)
- added REF**: PinHeader_1x04_P2.54mm_Vertical, Connector_PinHeader_2.54mm:PinHeader_1x04_P2.54mm_Vertical, F.Cu at (341.9, 83.7)
- added REF**: Stabilizer_Cherry_MX_2.00u, PCM_Mounting_Keyboard_Stabilizer:Stabilizer_Cherry_MX_2.00u, F.Cu at (72.5, 125.1)
- added REF**: PinHeader_1x04_P2.54mm_Vertical, Connector_PinHeader_2.54mm:PinHeader_1x04_P2.54mm_Vertical, F.Cu at (90.2, 37.6)
- added REF**: ConnectorMicromatch-4, ConnectorMicromatch-4, F.Cu at (338.5, 87.5)
- added REF**: ConnectorMicromatch-4, ConnectorMicromatch-4, F.Cu at (292.0, 41.0)
- added REF**: ConnectorMicromatch-4, ConnectorMicromatch-4, B.Cu at (338.5, 112.5)
- added REF**: ConnectorMicromatch-4, ConnectorMicromatch-4, B.Cu at (338.5, 87.5)
- added REF**: PinHeader_1x04_P2.54mm_Vertical, Connector_PinHeader_2.54mm:PinHeader_1x04_P2.54mm_Vertical, F.Cu at (341.9, 108.7)
- added REF**: ConnectorMicromatch-4, ConnectorMicromatch-4, B.Cu at (267.0, 41.0)
- added REF**: ConnectorMicromatch-4, ConnectorMicromatch-4, B.Cu at (94.0, 41.0)
- added REF**: ConnectorMicromatch-4, ConnectorMicromatch-4, B.Cu at (292.0, 41.0)
- added REF**: ConnectorMicromatch-4, ConnectorMicromatch-4, B.Cu at (119.0, 41.0)
- added REF**: Stabilizer_Cherry_MX_2.00u, PCM_Mounting_Keyboard_Stabilizer:Stabilizer_Cherry_MX_2.00u, F.Cu at (315.4, 106.0)
- added REF**: PinHeader_1x04_P2.54mm_Vertical, Connector_PinHeader_2.54mm:PinHeader_1x04_P2.54mm_Vertical, F.Cu at (263.2, 37.6)
- added REF**: Stabilizer_Cherry_MX_2.00u, PCM_Mounting_Keyboard_Stabilizer:Stabilizer_Cherry_MX_2.00u, F.Cu at (317.8, 68.8)
- added REF**: ConnectorMicromatch-4, ConnectorMicromatch-4, F.Cu at (119.0, 41.0)
- added REF**: PinHeader_1x04_P2.54mm_Vertical, Connector_PinHeader_2.54mm:PinHeader_1x04_P2.54mm_Vertical, F.Cu at (288.2, 37.6)
- added REF**: Stabilizer_Cherry_MX_2.00u, PCM_Mounting_Keyboard_Stabilizer:Stabilizer_Cherry_MX_2.00u, F.Cu at (310.6, 125.1)
- added REF**: ConnectorMicromatch-4, ConnectorMicromatch-4, F.Cu at (338.5, 112.5)
- added SW2: SW_Push, random-keyboard-parts.pretty-master:SKQG-1155865, B.Cu at (201.2, 116.0)
- added U2: SL2.1A, SL2.1A:SO16, B.Cu at (177.2, 54.2)
- added U4: XC6206PxxxMR, Package_TO_SOT_SMD:SOT-23-3, B.Cu at (211.0, 117.1)
- added U5: USBLC6-2SC6, Package_TO_SOT_SMD:SOT-23-6, B.Cu at (267.0, 52.6)
- added U6: STM32F072CBTx, Package_QFP:LQFP-48_7x7mm_P0.5mm, B.Cu at (207.0, 141.7)
- added U7: USBLC6-2SC6, Package_TO_SOT_SMD:SOT-23-6, B.Cu at (321.3, 96.5)
- added U8: USBLC6-2SC6, Package_TO_SOT_SMD:SOT-23-6, B.Cu at (94.1, 54.1)
- added mouse-bite-3mm-slot: VAL**, Panelization.pretty-master:mouse-bite-3mm-slot, F.Cu at (335.4, 100.0)
- added mouse-bite-3mm-slot: VAL**, Panelization.pretty-master:mouse-bite-3mm-slot, F.Cu at (106.5, 44.1)
- added mouse-bite-3mm-slot: VAL**, Panelization.pretty-master:mouse-bite-3mm-slot, F.Cu at (279.5, 44.1)
- C4: value 0.1uF -> 100nF; footprint Capacitor_SMD:C_0805_2012Metric -> Capacitor_SMD:C_0402_1005Metric; moved to B.Cu
- C5: value 10uF -> 1uF; footprint Capacitor_SMD:C_0805_2012Metric -> Capacitor_SMD:C_0402_1005Metric; moved to B.Cu
- C6: value 22pF -> 1uF; footprint Capacitor_SMD:C_0805_2012Metric -> Capacitor_SMD:C_0402_1005Metric; moved to B.Cu
- C7: value 22pF -> 100nF; footprint Capacitor_SMD:C_0805_2012Metric -> Capacitor_SMD:C_0402_1005Metric; moved to B.Cu
- J1, R5, R6: moved to B.Cu
- MX1, MX10, MX11, MX12, MX13, MX14, MX15, MX16, MX17, MX18, MX19, MX2, MX20, MX21, MX22, MX23, MX24, MX25, MX26, MX27, MX28, MX29, MX3, MX30, MX31, MX32, MX33, MX34, MX35, MX36, MX37, MX38, MX39, MX4, MX40, MX41, MX42, MX43, MX44, MX45, MX46, MX47, MX48, MX49, MX5, MX50, MX51, MX52, MX53, MX54, MX55, MX56, MX57, MX58, MX59, MX6, MX60, MX61, MX7, MX8, MX9: footprint keyswitches.pretty-master:Kailh_socket_MX -> PCM_marbastlib-mx:SW_MX_HS_CPG151101S11_1u; moved to B.Cu
- U1: value ATmega32U4-A -> USBLC6-2SC6; footprint Package_QFP:TQFP-44_10x10mm_P0.8mm -> Package_TO_SOT_SMD:SOT-23-6; moved to B.Cu
- moved D29 227.0 mm to (75.3, 110.9)
- moved D30 224.7 mm to (101.5, 110.9)
- moved D19 118.6 mm to (153.9, 91.8)
- moved D20 113.5 mm to (173.0, 91.8)
- moved C4 89.0 mm to (207.1, 147.8), turned to -90 degrees
- moved U1 81.6 mm to (193.5, 57.0), turned to 90 degrees
- moved D22 77.3 mm to (211.1, 91.8)
- moved D25 77.3 mm to (268.2, 91.8)
- moved D26 77.3 mm to (287.3, 91.8)
- moved D21 77.3 mm to (192.0, 91.8)
- moved D23 77.3 mm to (230.1, 91.8)
- moved D24 77.3 mm to (249.2, 91.8)
- moved D27 77.3 mm to (306.3, 91.8)
- moved D28 76.8 mm to (324.9, 92.1), turned to 45 degrees
- moved C7 65.7 mm to (209.8, 147.8), turned to 90 degrees
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Connections:
- C4 pad 1: +5V -> /NRST
- C5 pad 1: +5V -> Net-(U4-VI)
- C6 pad 1: GND -> +3.3V
- C6 pad 2: Net-(U1-XTAL1) -> GND
- C7 pad 2: Net-(U1-XTAL2) -> +3.3V
- D19 pad 1: ROW2 -> ROW1
- D20 pad 1: ROW2 -> ROW1
- D29 pad 1: ROW1 -> ROW2
- D30 pad 1: ROW1 -> ROW2
- J1 pad A4: +5V -> Net-(F2-Pad1)
- J1 pad A9: +5V -> Net-(F2-Pad1)
- J1 pad B4: +5V -> Net-(F2-Pad1)
- J1 pad B9: +5V -> Net-(F2-Pad1)
- MX19 pad 2: Net-(D21-A) -> Net-(D19-A)
- MX20 pad 2: Net-(D22-A) -> Net-(D20-A)
- MX21 pad 2: Net-(D23-A) -> Net-(D21-A)
- MX22 pad 2: Net-(D24-A) -> Net-(D22-A)
- MX23 pad 2: Net-(D25-A) -> Net-(D23-A)
- MX24 pad 2: Net-(D26-A) -> Net-(D24-A)
- MX25 pad 2: Net-(D27-A) -> Net-(D25-A)
- MX26 pad 2: Net-(D28-A) -> Net-(D26-A)
- MX27 pad 2: Net-(D29-A) -> Net-(D27-A)
- MX28 pad 2: Net-(D30-A) -> Net-(D28-A)
- MX29 pad 2: Net-(D19-A) -> Net-(D29-A)
- MX30 pad 2: Net-(D20-A) -> Net-(D30-A)
- R5 pad 2: Net-(J1-CC2) -> Net-(J1-CC1)
- R6 pad 2: Net-(J1-CC1) -> Net-(J1-CC2)
- U1 pad 1: unconnected-(U1-PE6-Pad1) -> /USB_Hub/ESD+
- U1 pad 2: +5V -> GND
- U1 pad 3: Net-(U1-D-) -> /USB_Hub/ESD-
- U1 pad 4: Net-(U1-D+) -> D-
- U1 pad 5: GND -> VBUS
- U1 pad 6: Net-(U1-UCAP) -> D+
Routing:
- net VBUS: track 0.00 -> 430.4 mm, vias 0 -> 8
- net ROW4: track 491.2 -> 280.4 mm, vias 8 -> 0
- net ROW3: track 467.2 -> 259.3 mm, vias 12 -> 4
- net D2+: track 0.00 -> 192.6 mm, vias 0 -> 2
- net D2-: track 0.00 -> 189.7 mm, vias 0 -> 4
- net ROW2: track 455.1 -> 290.8 mm, vias 13 -> 4
- net (no net): track 0.00 -> 149.5 mm
- net ROW1: track 441.1 -> 311.7 mm, vias 14 -> 4
- net COL12: track 79.2 -> 196.0 mm
- net D3-: track 0.00 -> 102.4 mm, vias 0 -> 2
- net D3+: track 0.00 -> 102.4 mm, vias 0 -> 2
- net D4+: track 0.00 -> 98.6 mm
- net D4-: track 0.00 -> 98.1 mm, vias 0 -> 2
- net D1+: track 0.00 -> 88.4 mm, vias 0 -> 1
- net D1-: track 0.00 -> 88.4 mm, vias 0 -> 1
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- added copper zone on B.Cu, net GND
- removed copper zone on B.Cu, net +5V
Other:
- board size 300 x 140 mm -> 296.4 x 123.4 mm
- board text added: "JLCJLCJLCJLC"
- board text added: "MODULE 1"
- board text added: "MODULE 2"
- board text added: "MODULE 3"
- board text added: "SN:"
- board text added: "SVRD60"
- board text added: "github.com/aKempista"
