File: CustomKeyboard.kicad_sch (KiCad schematic)
At the start: 18 parts, among them J1 USB_C_Receptacle_USB2.0_16P, J2 Conn_01x04, SW1 SW_Push, U1 ATmega32U4-A, Y1 16MHz

Commit message: many things changed
Parts:
- removed C1: 1uF, Capacitor_SMD:C_0805_2012Metric, symbol Device:C_Small
- removed C2, C3: 0.1uF, Capacitor_SMD:C_0805_2012Metric, symbol Device:C_Small
- removed J1: USB_C_Receptacle_USB2.0_16P, Connector_USB:USB_C_Receptacle_GCT_USB4105-xx-A_16P_TopMnt_Horizontal, symbol Connector:USB_C_Receptacle_USB2.0_16P
- removed J2: Conn_01x04, Connector_PinHeader_2.54mm:PinHeader_1x04_P2.54mm_Vertical, symbol Connector_Generic:Conn_01x04
- removed R1, R4: 10k, Resistor_SMD:R_0805_2012Metric, symbol Device:R_Small
- removed R2, R3: 22, Resistor_SMD:R_0805_2012Metric, symbol Device:R_Small
- removed R5, R6: 5.11k, Resistor_SMD:R_0805_2012Metric, symbol Device:R_Small
- removed SW1: SW_Push, random-keyboard-parts.pretty-master:SKQG-1155865, symbol Switch:SW_Push
- removed U1: ATmega32U4-A, Package_QFP:TQFP-44_10x10mm_P0.8mm, symbol MCU_Microchip_ATmega:ATmega32U4-A
- removed Y1: 16MHz, Crystal:Crystal_SMD_3225-4Pin_3.2x2.5mm, symbol Device:Crystal_GND24_Small
- added C19, C21, C24: 100nF, Capacitor_SMD:C_0402_1005Metric, symbol Device:C_Small
- added C20, C25: 4.7uF, Capacitor_SMD:C_0402_1005Metric, symbol Device:C_Small
- added C22: 10nF, Capacitor_SMD:C_0402_1005Metric, symbol Device:C_Small
- added C23: 1uF, Capacitor_SMD:C_0402_1005Metric, symbol Device:C_Small
- added F1: 500mA, Fuse:Fuse_0603_1608Metric, symbol Device:Fuse_Small
- added R10: 10k, Resistor_SMD:R_0402_1005Metric, symbol Device:R_Small
- added SW2: SW_Push, random-keyboard-parts.pretty-master:SKQG-1155865, symbol Switch:SW_Push
- added U4: XC6206PxxxMR, Package_TO_SOT_SMD:SOT-23-3, symbol Regulator_Linear:XC6206PxxxMR
- added U6: STM32F072CBTx, Package_QFP:LQFP-48_7x7mm_P0.5mm, symbol MCU_ST_STM32F0:STM32F072CBTx
- C4: value 0.1uF -> 100nF; footprint Capacitor_SMD:C_0805_2012Metric -> Capacitor_SMD:C_0402_1005Metric; LCSC (none) -> C307331
- C5: value 10uF -> 1uF; footprint Capacitor_SMD:C_0805_2012Metric -> Capacitor_SMD:C_0402_1005Metric; LCSC (none) -> C52923
- C6: value 22pF -> 1uF; footprint Capacitor_SMD:C_0805_2012Metric -> Capacitor_SMD:C_0402_1005Metric; LCSC (none) -> C52923
- C7: value 22pF -> 100nF; footprint Capacitor_SMD:C_0805_2012Metric -> Capacitor_SMD:C_0402_1005Metric; LCSC (none) -> C307331; MPN (none) -> CL05B104KB54PNC
Connections:
- net COL0: now also U6.25 (PB12)
- net COL1: now also U6.26 (PB13)
- net COL10: now also U6.40 (PB4)
- net COL11: now also U6.41 (PB5)
- net COL12: now also U6.42 (PB6)
- net COL13: now also U6.43 (PB7)
- net COL2: now also U6.27 (PB14)
- net COL3: now also U6.28 (PB15)
- net COL4: now also U6.29 (PA8)
- net COL5: now also U6.30 (PA9)
- net COL6: now also U6.31 (PA10)
- net COL7: now also U6.37 (PA14)
- net COL8: now also U6.38 (PA15)
- net COL9: now also U6.39 (PB3)
- net GND: now also C6.2, C19.1, C20.1, C21.1, C22.1, C23.1, C24.1, C25.1, R10.1, U4.1 (GND), U6.23 (VSS), U6.35 (VSS), U6.47 (VSS), U6.8 (VSSA); no longer C6.1
- net ROW1: now also U6.21 (PB10)
- net ROW2: now also U6.20 (PB2)
- net ROW3: now also U6.19 (PB1)
- net ROW4: now also U6.18 (PB0)
- net +3.3V: now reaches C7.2
- net +3.3V: now also C6.1, C19.2, C20.2, C21.2, C22.2, C23.2, C24.2, C25.2, SW2.1, U4.2 (VO), U6.1 (VBAT), U6.24 (VDD), U6.36 (VDDIO2), U6.48 (VDD), U6.9 (VDDA)
- net +5V: no longer names the net of C5.1
- net +5V: now also F1.1, U4.3 (VI); no longer C4.1
- new net A0: U6.10 (PA0)
- new net A1: U6.11 (PA1)
- new net A13: U6.34 (PA13)
- new net A2: U6.12 (PA2)
- new net A3: U6.13 (PA3)
- new net A4: U6.14 (PA4)
- new net A5: U6.15 (PA5)
- new net A6: U6.16 (PA6)
- new net A7: U6.17 (PA7)
- new net B8: U6.45 (PB8)
- new net B9: U6.46 (PB9)
- new net BOOT0: R10.2, SW2.2, U6.44 (BOOT0)
- new net C13: U6.2 (PC13)
- new net C14: U6.3 (PC14)
- new net C15: U6.4 (PC15)
- new net D4+: U6.33 (PA12)
- new net D4-: U6.32 (PA11)
- new net F0: U6.5 (PF0)
- new net F1: U6.6 (PF1)
- new net NRST: C4.1, U6.7 (NRST)
- new net ROW0: U6.22 (PB11)
- new net VBUS: F1.2
- no-connect marks 2 -> 0
