File: SwitchMatrix.kicad_sch (KiCad schematic)
At the start: 122 parts

Commit message: many things changed
Parts:
- MX1, MX61: footprint keyswitches.pretty-master:Kailh_socket_MX -> PCM_marbastlib-mx:SW_MX_HS_CPG151101S11_1u
- MX10: renamed from MX41; footprint keyswitches.pretty-master:Kailh_socket_MX -> PCM_marbastlib-mx:SW_MX_HS_CPG151101S11_1u
- MX11: renamed from MX46; footprint keyswitches.pretty-master:Kailh_socket_MX -> PCM_marbastlib-mx:SW_MX_HS_CPG151101S11_1u
- MX12: renamed from MX51; footprint keyswitches.pretty-master:Kailh_socket_MX -> PCM_marbastlib-mx:SW_MX_HS_CPG151101S11_1u
- MX13: renamed from MX55; footprint keyswitches.pretty-master:Kailh_socket_MX -> PCM_marbastlib-mx:SW_MX_HS_CPG151101S11_1u
- MX14: renamed from MX57; footprint keyswitches.pretty-master:Kailh_socket_MX -> PCM_marbastlib-mx:SW_MX_HS_CPG151101S11_1u
- MX15: renamed from MX2; footprint keyswitches.pretty-master:Kailh_socket_MX -> PCM_marbastlib-mx:SW_MX_HS_CPG151101S11_1u
- MX16: renamed from MX7; footprint keyswitches.pretty-master:Kailh_socket_MX -> PCM_marbastlib-mx:SW_MX_HS_CPG151101S11_1u
- MX17: renamed from MX12; footprint keyswitches.pretty-master:Kailh_socket_MX -> PCM_marbastlib-mx:SW_MX_HS_CPG151101S11_1u
- MX18: renamed from MX17; footprint keyswitches.pretty-master:Kailh_socket_MX -> PCM_marbastlib-mx:SW_MX_HS_CPG151101S11_1u
- MX19: renamed from MX21; footprint keyswitches.pretty-master:Kailh_socket_MX -> PCM_marbastlib-mx:SW_MX_HS_CPG151101S11_1u
- MX2: renamed from MX6; footprint keyswitches.pretty-master:Kailh_socket_MX -> PCM_marbastlib-mx:SW_MX_HS_CPG151101S11_1u
- MX20: renamed from MX25; footprint keyswitches.pretty-master:Kailh_socket_MX -> PCM_marbastlib-mx:SW_MX_HS_CPG151101S11_1u
- MX21: renamed from MX30; footprint keyswitches.pretty-master:Kailh_socket_MX -> PCM_marbastlib-mx:SW_MX_HS_CPG151101S11_1u
- MX22: renamed from MX34; footprint keyswitches.pretty-master:Kailh_socket_MX -> PCM_marbastlib-mx:SW_MX_HS_CPG151101S11_1u
- MX23: renamed from MX38; footprint keyswitches.pretty-master:Kailh_socket_MX -> PCM_marbastlib-mx:SW_MX_HS_CPG151101S11_1u
- MX24: renamed from MX42; footprint keyswitches.pretty-master:Kailh_socket_MX -> PCM_marbastlib-mx:SW_MX_HS_CPG151101S11_1u
- MX25: renamed from MX47; footprint keyswitches.pretty-master:Kailh_socket_MX -> PCM_marbastlib-mx:SW_MX_HS_CPG151101S11_1u
- MX26: renamed from MX52; footprint keyswitches.pretty-master:Kailh_socket_MX -> PCM_marbastlib-mx:SW_MX_HS_CPG151101S11_1u
- MX27: renamed from MX56; footprint keyswitches.pretty-master:Kailh_socket_MX -> PCM_marbastlib-mx:SW_MX_HS_CPG151101S11_1u
- MX28: renamed from MX58; footprint keyswitches.pretty-master:Kailh_socket_MX -> PCM_marbastlib-mx:SW_MX_HS_CPG151101S11_1u
- MX29: renamed from MX3; footprint keyswitches.pretty-master:Kailh_socket_MX -> PCM_marbastlib-mx:SW_MX_HS_CPG151101S11_1u
- MX3: renamed from MX11; footprint keyswitches.pretty-master:Kailh_socket_MX -> PCM_marbastlib-mx:SW_MX_HS_CPG151101S11_1u
- MX30: renamed from MX8; footprint keyswitches.pretty-master:Kailh_socket_MX -> PCM_marbastlib-mx:SW_MX_HS_CPG151101S11_1u
- MX31: renamed from MX13; footprint keyswitches.pretty-master:Kailh_socket_MX -> PCM_marbastlib-mx:SW_MX_HS_CPG151101S11_1u
- MX32: renamed from MX18; footprint keyswitches.pretty-master:Kailh_socket_MX -> PCM_marbastlib-mx:SW_MX_HS_CPG151101S11_1u
- MX33: renamed from MX22; footprint keyswitches.pretty-master:Kailh_socket_MX -> PCM_marbastlib-mx:SW_MX_HS_CPG151101S11_1u
- MX34: renamed from MX26; footprint keyswitches.pretty-master:Kailh_socket_MX -> PCM_marbastlib-mx:SW_MX_HS_CPG151101S11_1u
- MX35: renamed from MX31; footprint keyswitches.pretty-master:Kailh_socket_MX -> PCM_marbastlib-mx:SW_MX_HS_CPG151101S11_1u
- MX36: renamed from MX35; footprint keyswitches.pretty-master:Kailh_socket_MX -> PCM_marbastlib-mx:SW_MX_HS_CPG151101S11_1u
- MX37: renamed from MX39; footprint keyswitches.pretty-master:Kailh_socket_MX -> PCM_marbastlib-mx:SW_MX_HS_CPG151101S11_1u
- MX38: renamed from MX43; footprint keyswitches.pretty-master:Kailh_socket_MX -> PCM_marbastlib-mx:SW_MX_HS_CPG151101S11_1u
- MX39: renamed from MX48; footprint keyswitches.pretty-master:Kailh_socket_MX -> PCM_marbastlib-mx:SW_MX_HS_CPG151101S11_1u
- MX4: renamed from MX16; footprint keyswitches.pretty-master:Kailh_socket_MX -> PCM_marbastlib-mx:SW_MX_HS_CPG151101S11_1u
- MX40: renamed from MX53; footprint keyswitches.pretty-master:Kailh_socket_MX -> PCM_marbastlib-mx:SW_MX_HS_CPG151101S11_1u
- MX41: renamed from MX59; footprint keyswitches.pretty-master:Kailh_socket_MX -> PCM_marbastlib-mx:SW_MX_HS_CPG151101S11_1u
- MX42: renamed from MX4; footprint keyswitches.pretty-master:Kailh_socket_MX -> PCM_marbastlib-mx:SW_MX_HS_CPG151101S11_1u
- MX43: renamed from MX9; footprint keyswitches.pretty-master:Kailh_socket_MX -> PCM_marbastlib-mx:SW_MX_HS_CPG151101S11_1u
- MX44: renamed from MX14; footprint keyswitches.pretty-master:Kailh_socket_MX -> PCM_marbastlib-mx:SW_MX_HS_CPG151101S11_1u
- MX45: renamed from MX19; footprint keyswitches.pretty-master:Kailh_socket_MX -> PCM_marbastlib-mx:SW_MX_HS_CPG151101S11_1u
- MX46: renamed from MX23; footprint keyswitches.pretty-master:Kailh_socket_MX -> PCM_marbastlib-mx:SW_MX_HS_CPG151101S11_1u
- MX47: renamed from MX27; footprint keyswitches.pretty-master:Kailh_socket_MX -> PCM_marbastlib-mx:SW_MX_HS_CPG151101S11_1u
- MX48: renamed from MX32; footprint keyswitches.pretty-master:Kailh_socket_MX -> PCM_marbastlib-mx:SW_MX_HS_CPG151101S11_1u
- MX49: renamed from MX36; footprint keyswitches.pretty-master:Kailh_socket_MX -> PCM_marbastlib-mx:SW_MX_HS_CPG151101S11_1u
- MX5: renamed from MX20; footprint keyswitches.pretty-master:Kailh_socket_MX -> PCM_marbastlib-mx:SW_MX_HS_CPG151101S11_1u
- MX50: renamed from MX40; footprint keyswitches.pretty-master:Kailh_socket_MX -> PCM_marbastlib-mx:SW_MX_HS_CPG151101S11_1u
- MX51: renamed from MX44; footprint keyswitches.pretty-master:Kailh_socket_MX -> PCM_marbastlib-mx:SW_MX_HS_CPG151101S11_1u
- MX52: renamed from MX49; footprint keyswitches.pretty-master:Kailh_socket_MX -> PCM_marbastlib-mx:SW_MX_HS_CPG151101S11_1u
- MX53: renamed from MX60; footprint keyswitches.pretty-master:Kailh_socket_MX -> PCM_marbastlib-mx:SW_MX_HS_CPG151101S11_1u
- MX54: renamed from MX5; footprint keyswitches.pretty-master:Kailh_socket_MX -> PCM_marbastlib-mx:SW_MX_HS_CPG151101S11_1u
- MX55: renamed from MX10; footprint keyswitches.pretty-master:Kailh_socket_MX -> PCM_marbastlib-mx:SW_MX_HS_CPG151101S11_1u
- MX56: renamed from MX15; footprint keyswitches.pretty-master:Kailh_socket_MX -> PCM_marbastlib-mx:SW_MX_HS_CPG151101S11_1u
- MX57: renamed from MX28; footprint keyswitches.pretty-master:Kailh_socket_MX -> PCM_marbastlib-mx:SW_MX_HS_CPG151101S11_1u
- MX58: renamed from MX45; footprint keyswitches.pretty-master:Kailh_socket_MX -> PCM_marbastlib-mx:SW_MX_HS_CPG151101S11_1u
- MX59: renamed from MX50; footprint keyswitches.pretty-master:Kailh_socket_MX -> PCM_marbastlib-mx:SW_MX_HS_CPG151101S11_1u
- MX6: renamed from MX24; footprint keyswitches.pretty-master:Kailh_socket_MX -> PCM_marbastlib-mx:SW_MX_HS_CPG151101S11_1u
- MX60: renamed from MX54; footprint keyswitches.pretty-master:Kailh_socket_MX -> PCM_marbastlib-mx:SW_MX_HS_CPG151101S11_1u
- MX7: renamed from MX29; footprint keyswitches.pretty-master:Kailh_socket_MX -> PCM_marbastlib-mx:SW_MX_HS_CPG151101S11_1u
- MX8: renamed from MX33; footprint keyswitches.pretty-master:Kailh_socket_MX -> PCM_marbastlib-mx:SW_MX_HS_CPG151101S11_1u
- MX9: renamed from MX37; footprint keyswitches.pretty-master:Kailh_socket_MX -> PCM_marbastlib-mx:SW_MX_HS_CPG151101S11_1u
- renumbered D41 to D10, D46 to D11, D51 to D12, D55 to D13, D57 to D14, D2 to D15, D7 to D16, D12 to D17, D17 to D18, D21 to D19, D6 to D2, D25 to D20, D30 to D21, D34 to D22, D38 to D23, D42 to D24, D47 to D25, D52 to D26, D56 to D27, D58 to D28, D3 to D29, D11 to D3, D8 to D30, D13 to D31, D18 to D32, D22 to D33, D26 to D34, D31 to D35, D35 to D36, D39 to D37, D43 to D38, D48 to D39, D16 to D4, D53 to D40, D59 to D41, D4 to D42, D9 to D43, D14 to D44, D19 to D45, D23 to D46, D27 to D47, D32 to D48, D36 to D49, D20 to D5, D40 to D50, D44 to D51, D49 to D52, D60 to D53, D5 to D54, D10 to D55, D15 to D56, D28 to D57, D45 to D58, D50 to D59, D24 to D6, D54 to D60, D29 to D7, D33 to D8, D37 to D9
